File: driverTest2/driverTest2.kicad_pcb (KiCad board)
At the start: 2 copper layers, 35 x 18 mm, 9 parts, among them J1 INPUT, J2 LED_OUTPUT, U1 RT8498

Commit message: Commit last minute changes
Parts:
- moved C2 0.41 mm to (145.6, 82.5)
Other:
- board size 35 x 18 mm -> 39 x 18 mm
- board text added: "LED+"
- board text added: "LED-"
- board text added: "RT8498 breakout Jan Mrázek 08/2020 v0.1"
- board text added: "VCC GND DCTL ACTL"
