File: driverTest2/driverTest2.sch (KiCad schematic (older format))
At the start: 9 parts

Commit message: Commit last minute changes
Parts:
- gave numbers to parts that had none: 9
Changed lines of the file:
@@
 $EndDescr
 $Comp
-L headlamp:RT8498 U?
+L headlamp:RT8498 U1
 U 1 1 5F2FABD8
 P 6100 3250
-F 0 "U?" H 6100 3525 50  0000 C CNN
+F 0 "U1" H 6100 3525 50  0000 C CNN
 F 1 "RT8498" H 6100 3434 50  0000 C CNN
 F 2 "Package_TO_SOT_SMD:SOT-23-6_Handsoldering" H 6100 3500 50  0001 C CNN
@@
 $EndComp
 $Comp
-L Device:L L?
+L Device:L L1
 U 1 1 5F2FB2D2
 P 5400 2800
-F 0 "L?" V 5590 2800 50  0000 C CNN
+F 0 "L1" V 5590 2800 50  0000 C CNN
 F 1 "SRU1038-100Y" V 5499 2800 50  0000 C CNN
 F 2 "Inductor_SMD:L_Bourns-SRU1028_10.0x10.0mm" H 5400 2800 50  0001 C CNN
@@
 $EndComp
 $Comp
-L Device:D D?
+L Device:D D1
 U 1 1 5F2FBAC0
 P 6100 2800
-F 0 "D?" H 6100 2583 50  0000 C CNN
+F 0 "D1" H 6100 2583 50  0000 C CNN
 F 1 "FML340A-W" H 6100 2674 50  0000 C CNN
 F 2 "headlamp:DO-214AC" H 6100 2800 50  0001 C CNN
@@
 $EndComp
 $Comp
-L Device:C C?
+L Device:C C2
 U 1 1 5F2FC1DF
 P 7800 3350
-F 0 "C?" H 7915 3396 50  0000 L CNN
+F 0 "C2" H 7915 3396 50  0000 L CNN
 F 1 "100n" H 7915 3305 50  0000 L CNN
 F 2 "Capacitor_SMD:C_0603_1608Metric_Pad1.05x0.95mm_HandSolder" H 7838 3200 50  0001 C CNN
@@
 $EndComp
 $Comp
-L Device:C C?
+L Device:C C3
 U 1 1 5F2FCDFF
 P 8250 3050
-F 0 "C?" H 8135 3004 50  0000 R CNN
+F 0 "C3" H 8135 3004 50  0000 R CNN
 F 1 "470n" H 8135 3095 50  0000 R CNN
 F 2 "Capacitor_SMD:C_0603_1608Metric_Pad1.05x0.95mm_HandSolder" H 8288 2900 50  0001 C CNN
@@
 $EndComp
 $Comp
-L Device:R R?
+L Device:R R1
 U 1 1 5F2FD342
 P 7000 3350
-F 0 "R?" H 7070 3396 50  0000 L CNN
+F 0 "R1" H 7070 3396 50  0000 L CNN
 F 1 "KDV12FR050ET" H 7070 3305 50  0000 L CNN
 F 2 "Resistor_SMD:R_1206_3216Metric" V 6930 3350 50  0001 C CNN
@@
 	7000 3200 7800 3200
 $Comp
-L power:GND #PWR?
+L power:GND #PWR08
 U 1 1 5F2FFF48
 P 7800 3500
-F 0 "#PWR?" H 7800 3250 50  0001 C CNN
+F 0 "#PWR08" H 7800 3250 50  0001 C CNN
 F 1 "GND" H 7805 3327 50  0000 C CNN
 F 2 "" H 7800 3500 50  0001 C CNN
@@
 DCTL
 $Comp
-L Device:C C?
+L Device:C C1
 U 1 1 5F301AF2
 P 5500 3600
-F 0 "C?" H 5615 3646 50  0000 L CNN
+F 0 "C1" H 5615 3646 50  0000 L CNN
 F 1 "10n" H 5615 3555 50  0000 L CNN
 F 2 "Capacitor_SMD:C_0603_1608Metric_Pad1.05x0.95mm_HandSolder" H 5538 3450 50  0001 C CNN
@@
 Connection ~ 5500 3400
 $Comp
-L power:GND #PWR?
+L power:GND #PWR02
 U 1 1 5F3026CE
 P 5500 3750
-F 0 "#PWR?" H 5500 3500 50  0001 C CNN
+F 0 "#PWR02" H 5500 3500 50  0001 C CNN
 F 1 "GND" H 5505 3577 50  0000 C CNN
 F 2 "" H 5500 3750 50  0001 C CNN
@@
 $EndComp
 $Comp
-L power:GND #PWR?
+L power:GND #PWR05
 U 1 1 5F302A19
 P 6100 3600
-F 0 "#PWR?" H 6100 3350 50  0001 C CNN
+F 0 "#PWR05" H 6100 3350 50  0001 C CNN
 F 1 "GND" H 6105 3427 50  0000 C CNN
 F 2 "" H 6100 3600 50  0001 C CNN
@@
 ACTL
 $Comp
-L power:VCC #PWR?
+L power:VCC #PWR01
 U 1 1 5F303362
 P 4700 2800
-F 0 "#PWR?" H 4700 2650 50  0001 C CNN
+F 0 "#PWR01" H 4700 2650 50  0001 C CNN
 F 1 "VCC" V 4715 2927 50  0000 L CNN
 F 2 "" H 4700 2800 50  0001 C CNN
@@
 Connection ~ 4800 2800
 $Comp
-L Connector_Generic:Conn_02x02_Odd_Even J?
+L Connector_Generic:Conn_02x02_Odd_Even J2
 U 1 1 5F312023
 P 7500 1350
-F 0 "J?" H 7550 1567 50  0000 C CNN
+F 0 "J2" H 7550 1567 50  0000 C CNN
 F 1 "LED_OUTPUT" H 7550 1476 50  0000 C CNN
 F 2 "Connector_PinHeader_2.54mm:PinHeader_2x02_P2.54mm_Vertical" H 7500 1350 50  0001 C CNN
@@
 LED-
 $Comp
-L Connector_Generic:Conn_02x04_Odd_Even J?
+L Connector_Generic:Conn_02x04_Odd_Even J1
 U 1 1 5F313B48
 P 5850 1350
-F 0 "J?" H 5900 1667 50  0000 C CNN
+F 0 "J1" H 5900 1667 50  0000 C CNN
 F 1 "INPUT" H 5900 1576 50  0000 C CNN
 F 2 "Connector_PinHeader_2.54mm:PinHeader_2x04_P2.54mm_Vertical" H 5850 1350 50  0001 C CNN
@@
 $EndComp
 $Comp
-L power:VCC #PWR?
+L power:VCC #PWR03
 U 1 1 5F314AA7
 P 5650 1250
-F 0 "#PWR?" H 5650 1100 50  0001 C CNN
+F 0 "#PWR03" H 5650 1100 50  0001 C CNN
 F 1 "VCC" V 5665 1377 50  0000 L CNN
 F 2 "" H 5650 1250 50  0001 C CNN
@@
 $EndComp
 $Comp
-L power:VCC #PWR?
+L power:VCC #PWR06
 U 1 1 5F314EF3
 P 6150 1250
-F 0 "#PWR?" H 6150 1100 50  0001 C CNN
+F 0 "#PWR06" H 6150 1100 50  0001 C CNN
 F 1 "VCC" V 6165 1378 50  0000 L CNN
 F 2 "" H 6150 1250 50  0001 C CNN
@@
 $EndComp
 $Comp
-L power:GND #PWR?
+L power:GND #PWR04
 U 1 1 5F31533B
 P 5650 1350
-F 0 "#PWR?" H 5650 1100 50  0001 C CNN
+F 0 "#PWR04" H 5650 1100 50  0001 C CNN
 F 1 "GND" V 5655 1222 50  0000 R CNN
 F 2 "" H 5650 1350 50  0001 C CNN
@@
 $EndComp
 $Comp
-L power:GND #PWR?
+L power:GND #PWR07
 U 1 1 5F31575B
 P 6150 1350
-F 0 "#PWR?" H 6150 1100 50  0001 C CNN
+F 0 "#PWR07" H 6150 1100 50  0001 C CNN
 F 1 "GND" V 6155 1222 50  0000 R CNN
 F 2 "" H 6150 1350 50  0001 C CNN
