File: MP8859-breakout/MP8859-breakout.kicad_pcb (KiCad board)
At the start: 2 copper layers, 45 x 18 mm, 25 parts, among them J1 IO, J2 LED, U1 MP8859

Commit message: Tweak assembly data
Parts:
- added H1: MountingHole, MountingHole:MountingHole_2.2mm_M2, F.Cu at (153.0, 54.0)
- added H2: MountingHole, MountingHole:MountingHole_2.2mm_M2, F.Cu at (192.0, 66.0)
- added H3: MountingHole, MountingHole:MountingHole_2.2mm_M2, F.Cu at (192.0, 54.0)
- added H4: MountingHole, MountingHole:MountingHole_2.2mm_M2, F.Cu at (153.0, 66.0)
- moved J2 1.70 mm to (192.3, 60.8)
Other:
- outline, holes or cut-outs redrawn
- board text added: "GND VCC SCL SDA ALR"
- board text added: "LED+"
- board text added: "LED-"
- board text added: "MP8859 Breakout Jan Mrázek 08/20 v0.1"
