File: driverTest1/driverTest1.kicad_pcb (KiCad board)
At the start: 2 copper layers, 35 parts, among them J1 LED_OUT, J2 INPUT, U1 TPS63020, U2 MCP602, U3 XC6206P332MR

Commit message: Add new schema
Parts:
- removed C14: C, Capacitor_SMD:C_0402_1005Metric
- added NT1: SenseTie, NetTie:NetTie-2_SMD_Pad0.5mm, F.Cu at (154.1, 69.8)
- added Q1: 2N7002, Package_TO_SOT_SMD:SOT-23, F.Cu at (138.3, 68.7)
- added Q2: 2N7002, Package_TO_SOT_SMD:SOT-23, F.Cu at (146.8, 58.5)
- added R13: 120k, Resistor_SMD:R_0603_1608Metric, F.Cu at (154.6, 62.5)
- added R14: 30k, Resistor_SMD:R_0603_1608Metric, F.Cu at (159.0, 60.0)
- added R15: 30k, Resistor_SMD:R_0603_1608Metric, F.Cu at (150.6, 67.5)
- added R16: 120k, Resistor_SMD:R_0603_1608Metric, F.Cu at (154.6, 65.0)
- added R17: 120k, Resistor_SMD:R_0603_1608Metric, F.Cu at (158.6, 62.5)
- added R18: 51k, Resistor_SMD:R_0603_1608Metric, F.Cu at (150.6, 70.0)
- added R19: 1k8, Resistor_SMD:R_0603_1608Metric, F.Cu at (154.6, 67.5)
- added TP2: 3V3, TestPoint:TestPoint_THTPad_1.5x1.5mm_Drill0.7mm, F.Cu at (158.3, 65.5)
- added TP3: AmplifiedFeedback, TestPoint:TestPoint_THTPad_1.5x1.5mm_Drill0.7mm, F.Cu at (168.6, 65.0)
- C1, C10, C5: footprint Capacitor_SMD:C_0402_1005Metric -> Capacitor_SMD:C_0603_1608Metric
- C11: value C -> 220p; footprint Capacitor_SMD:C_0402_1005Metric -> Capacitor_SMD:C_0603_1608Metric
- C12: value C -> 1n5; footprint Capacitor_SMD:C_0402_1005Metric -> Capacitor_SMD:C_0603_1608Metric
- C13: value C -> 100n; footprint Capacitor_SMD:C_0402_1005Metric -> Capacitor_SMD:C_0603_1608Metric
- C8: value C -> 3n3; footprint Capacitor_SMD:C_0402_1005Metric -> Capacitor_SMD:C_0603_1608Metric
- L1: value 1u -> 1u5; footprint headlamp:MWSA0603 -> headlamp:MWSA0518
- R1: value 5m -> 20m; footprint Resistor_SMD:R_1206_3216Metric -> Resistor_SMD:R_0805_2012Metric
- R10: value R -> 3k3
- R11, R12, R6, R8: value R -> 30k
- R2, R3: value 10k -> 120k
- R4: value R -> 9k1
- R5: value R -> 91k
- R7: value R -> 120k
- R9: value R -> 51k
- TP1: value FB -> ChipFeedback; footprint TestPoint:TestPoint_THTPad_1.0x1.0mm_Drill0.5mm -> TestPoint:TestPoint_THTPad_1.5x1.5mm_Drill0.7mm
- U2: value MCP602 -> TPH2504-SR; footprint Package_SO:SOIC-8_3.9x4.9mm_P1.27mm -> Package_SO:SOIC-14_3.9x8.7mm_P1.27mm
- moved C8 34.5 mm to (155.0, 60.0)
- moved R10 33.3 mm to (159.0, 57.5)
- moved R4 33.3 mm to (155.0, 57.5)
- moved C13 29.8 mm to (151.0, 60.0)
- moved C11 27.6 mm to (151.0, 57.5)
- moved C12 25.1 mm to (142.5, 67.7)
- moved R9 24.0 mm to (146.5, 62.0)
- moved R8 23.0 mm to (150.6, 62.5)
- moved R5 21.5 mm to (146.5, 64.5)
- moved R7 21.5 mm to (146.6, 67.1)
- moved R6 20.9 mm to (142.5, 70.2)
- moved R12 19.8 mm to (150.6, 65.0)
- moved U2 19.1 mm to (140.3, 61.3)
- moved TP1 19.0 mm to (165.0, 65.0)
- moved R11 18.6 mm to (146.6, 69.6)
Connections:
- C12 pad 1: GND -> Net-(C12-Pad1)
- C12 pad 2: +3V3 -> Net-(C12-Pad2)
- C13 pad 1: Net-(C13-Pad1) -> +3V3
- C13 pad 2: DAC -> GND
- J2 pad 11: DAC -> FAST_DIM
- J2 pad 12: DAC -> FAST_DIM
- R1 pad 2: GND -> Net-(NT1-Pad1)
- R10 pad 1: GND -> Net-(Q1-Pad3)
- R10 pad 2: Net-(R10-Pad2) -> GND
- R11 pad 1: Net-(C13-Pad1) -> Net-(Q2-Pad2)
- R11 pad 2: Net-(C14-Pad1) -> Net-(R11-Pad2)
- R12 pad 1: PWM -> LED-
- R12 pad 2: Net-(C13-Pad1) -> Net-(R12-Pad2)
- R4 pad 1: Net-(R4-Pad1) -> Net-(C8-Pad2)
- R4 pad 2: Net-(C8-Pad2) -> PWM
- R5 pad 1: Net-(C11-Pad2) -> Net-(C12-Pad2)
- R5 pad 2: Net-(R4-Pad1) -> Net-(C8-Pad2)
- R6 pad 1: LED- -> Net-(C11-Pad2)
- R6 pad 2: Net-(R6-Pad2) -> Net-(C12-Pad2)
- R7 pad 1: DAC -> Net-(R7-Pad1)
- R7 pad 2: Net-(C11-Pad2) -> Net-(R7-Pad2)
- R8 pad 1: GND -> Net-(R7-Pad1)
- R8 pad 2: Net-(R6-Pad2) -> GND
- R9 pad 1: Net-(R10-Pad2) -> Net-(Q1-Pad3)
- R9 pad 2: DAC -> Net-(C12-Pad1)
- TP1 pad 1: Net-(R4-Pad1) -> Net-(R7-Pad2)
- U1 pad 3: Net-(C8-Pad2) -> Net-(R7-Pad2)
- U2 pad 1: Net-(R4-Pad1) -> Net-(R14-Pad1)
- U2 pad 2: Net-(R6-Pad2) -> Net-(R15-Pad2)
- U2 pad 3: Net-(C11-Pad2) -> Net-(R12-Pad2)
- U2 pad 4: GND -> +3V3
- U2 pad 5: Net-(R10-Pad2) -> Net-(Q2-Pad2)
- U2 pad 6: Net-(C14-Pad1) -> Net-(R7-Pad1)
- U2 pad 7: DAC -> Net-(R7-Pad2)
- U2 pad 8: +3V3 -> Net-(R11-Pad2)

Commit message: Draft first board layout
Parts:
- added H1: MountingHole, MountingHole:MountingHole_2.2mm_M2, F.Cu at (123.0, 38.0)
- added H2: MountingHole, MountingHole:MountingHole_2.2mm_M2, F.Cu at (152.0, 38.0)
- added H3: MountingHole, MountingHole:MountingHole_2.2mm_M2, F.Cu at (152.0, 62.0)
- added H4: MountingHole, MountingHole:MountingHole_2.2mm_M2, F.Cu at (123.0, 62.0)
- moved C3 49.2 mm to (129.0, 43.8), turned to 270 degrees
- moved C5 48.9 mm to (132.0, 43.8), turned to 270 degrees
- moved C6 48.5 mm to (142.8, 42.2), turned to 270 degrees
- moved R2 47.8 mm to (132.3, 48.0)
- moved C1 47.5 mm to (139.5, 46.8), turned to 180 degrees
- moved C2 47.3 mm to (127.4, 43.8), turned to 270 degrees
- moved U1 46.8 mm to (136.0, 45.0), turned to 90 degrees
- moved C10 46.3 mm to (141.3, 42.2), turned to 270 degrees
- moved C4 46.1 mm to (130.5, 43.8), turned to 270 degrees
- moved C7 45.6 mm to (144.3, 42.2), turned to 270 degrees
- moved C15 45.3 mm to (128.6, 56.0), turned to 180 degrees
- moved C16 43.7 mm to (130.6, 56.0)
- moved J1 41.8 mm to (150.0, 44.0)
- moved C9 40.5 mm to (145.9, 42.2), turned to 270 degrees
- moved L1 39.3 mm to (136.0, 39.4)
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Connections:
- U1 pad 13: Net-(C1-Pad2) -> +3V3
- U2 pad 1: Net-(R14-Pad1) -> Net-(R7-Pad2)
- U2 pad 12: Net-(C11-Pad2) -> Net-(R12-Pad2)
- U2 pad 13: Net-(C12-Pad1) -> Net-(R15-Pad2)
- U2 pad 14: Net-(C12-Pad1) -> Net-(R14-Pad1)
- U2 pad 2: Net-(R15-Pad2) -> Net-(R7-Pad1)
- U2 pad 3: Net-(R12-Pad2) -> Net-(Q2-Pad2)
- U2 pad 5: Net-(Q2-Pad2) -> Net-(C11-Pad2)
- U2 pad 6: Net-(R7-Pad1) -> Net-(C12-Pad1)
- U2 pad 7: Net-(R7-Pad2) -> Net-(C12-Pad1)
Routing:
- net +3V3: track 0.00 -> 50.9 mm, vias 0 -> 4
- net FAST_DIM: track 0.00 -> 39.7 mm
- net Net-(R7-Pad2): track 0.00 -> 28.9 mm, vias 0 -> 2
- net Net-(Q2-Pad2): track 0.00 -> 27.2 mm, vias 0 -> 1
- net PWM: track 0.00 -> 16.8 mm
- net POWER_GOOD: track 0.00 -> 16.2 mm, vias 0 -> 1
- net GND: track 0.00 -> 16.1 mm, vias 0 -> 79
- net Net-(Q1-Pad3): track 0.00 -> 15.8 mm, vias 0 -> 2
- net ENABLE: track 0.00 -> 14.5 mm, vias 0 -> 1
- net Net-(C8-Pad2): track 0.00 -> 14.1 mm
- net VCC: track 0.00 -> 13.7 mm
- net Net-(C12-Pad2): track 0.00 -> 7.18 mm
- net Net-(C12-Pad1): track 0.00 -> 5.79 mm
- net Net-(R14-Pad1): track 0.00 -> 5.61 mm
- net Net-(NT1-Pad1): track 0.00 -> 5.54 mm
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- added copper zone on B.Cu, net GND
- added copper zone on F.Cu, net GND
- added copper zone on F.Cu, net LED+
- added copper zone on F.Cu, net LED-
- added copper zone on F.Cu, net Net-(L1-Pad1)
- added copper zone on F.Cu, net Net-(L1-Pad2)
- added copper zone on F.Cu, net VCC
Other:
- board outline added: 35 x 30 mm

Commit message: Tweak assembly data
Parts:
- turned U1 to 180 degrees
