File: driverTest1/driverTest1.sch (KiCad schematic (older format))
At the start: 35 parts, among them J1 LED_OUT, J2 INPUT, U1 TPS63020, U2 MCP602, U3 XC6206P332MR

Commit message: Add routing note
Parts:
- added NT?: SenseTie, NetTie:NetTie-2_SMD_Pad0.5mm, symbol Device:Net-Tie_2
Connections:
- net GND: now also NT?.2; no longer R1.2, R8.1
- new net: NT?.1, R1.2, R8.1
Other:
- note added: "Connect these two grounds together first and then via a single point to the rest\nof the ground. The bottom ground should be connected directly to the pad of the\nsense resistor."
- moved on the sheet: R8
Changed lines of the file:
@@
 L power:GND #PWR0105
 U 1 1 5F1D53F5
-P 7850 1950
-F 0 "#PWR0105" H 7850 1700 50  0001 C CNN
-F 1 "GND" V 7855 1822 50  0000 R CNN
-F 2 "" H 7850 1950 50  0001 C CNN
-F 3 "" H 7850 1950 50  0001 C CNN
-	1    7850 1950
+P 8050 1950
+F 0 "#PWR0105" H 8050 1700 50  0001 C CNN
+F 1 "GND" V 8055 1822 50  0000 R CNN
+F 2 "" H 8050 1950 50  0001 C CNN
+F 3 "" H 8050 1950 50  0001 C CNN
+	1    8050 1950
 	0    -1   -1   0
 $EndComp
@@
 L Device:R R8
 U 1 1 5F1D8F6D
-P 7550 2400
-F 0 "R8" V 7450 2400 50  0000 C CNN
-F 1 "R" V 7550 2400 50  0000 C CNN
-F 2 "Resistor_SMD:R_0603_1608Metric" V 7480 2400 50  0001 C CNN
-F 3 "~" H 7550 2400 50  0001 C CNN
-	1    7550 2400
+P 7450 2400
+F 0 "R8" V 7350 2400 50  0000 C CNN
+F 1 "R" V 7450 2400 50  0000 C CNN
+F 2 "Resistor_SMD:R_0603_1608Metric" V 7380 2400 50  0001 C CNN
+F 3 "~" H 7450 2400 50  0001 C CNN
+	1    7450 2400
 	0    1    1    0
 $EndComp
@@
 	7250 1950 7100 1950
 Wire Wire Line
-	7400 2400 7250 2400
+	7300 2400 7250 2400
 Wire Wire Line
 	7250 2400 7250 2350
@@
 	8500 3200 8300 3200
 Wire Wire Line
-	8300 3200 8300 2600
-Wire Wire Line
-	8300 2600 8450 2600
+	8300 3200 8400 2600
+Wire Wire Line
+	8400 2600 8450 2600
 $Comp
 L Amplifier_Operational:MCP602 U2
@@
 	10050 1950 9550 1950
 Wire Wire Line
-	9250 1950 8300 1950
-Wire Wire Line
-	8300 1950 8300 2600
-Connection ~ 8300 2600
-Wire Wire Line
-	8300 2600 8100 2600
+	9250 1950 8400 1950
+Wire Wire Line
+	8400 1950 8400 2600
+Connection ~ 8400 2600
+Wire Wire Line
+	8400 2600 8100 2600
 Wire Wire Line
 	8100 2600 8100 3500
@@
 Text GLabel 2750 6050 2    50   Input ~ 0
 DAC
-Wire Wire Line
-	7600 1950 7850 1950
-$Comp
-L power:GND #PWR0131
-U 1 1 5F329A72
-P 7850 2400
-F 0 "#PWR0131" H 7850 2150 50  0001 C CNN
-F 1 "GND" V 7855 2272 50  0000 R CNN
-F 2 "" H 7850 2400 50  0001 C CNN
-F 3 "" H 7850 2400 50  0001 C CNN
-	1    7850 2400
-	0    -1   -1   0
-$EndComp
-Wire Wire Line
-	7850 2400 7700 2400
 $Comp
 L Connector:TestPoint TP1
@@
 Wire Wire Line
 	6300 2350 6300 2500
+Text Notes 7500 1550 0    50   ~ 0
+Connect these two grounds together first and then via a single point to the rest\nof the ground. The bottom ground should be connected directly to the pad of the\nsense resistor.
+$Comp
+L Device:Net-Tie_2 NT?
+U 1 1 5F3732B0
+P 7850 1950
+F 0 "NT?" H 7850 2131 50  0000 C CNN
+F 1 "SenseTie" H 7850 2040 50  0000 C CNN
+F 2 "NetTie:NetTie-2_SMD_Pad0.5mm" H 7850 1950 50  0001 C CNN
+F 3 "~" H 7850 1950 50  0001 C CNN
+	1    7850 1950
+	1    0    0    -1
+$EndComp
+Wire Wire Line
+	7600 2400 7600 1950
+Connection ~ 7600 1950
+Wire Wire Line
+	7600 1950 7750 1950
+Wire Wire Line
+	8050 1950 7950 1950
+Wire Notes Line
+	7500 2450 8350 2450
+Wire Notes Line
+	8350 2450 8350 1600
+Wire Notes Line
+	8350 1600 7500 1600
+Wire Notes Line
+	7500 1600 7500 2450
 $EndSCHEMATC

Commit message: Add new schema
Parts:
- removed C14: C, Capacitor_SMD:C_0402_1005Metric, symbol Device:C
- removed U2: MCP602, Package_SO:SOIC-8_3.9x4.9mm_P1.27mm, symbol Amplifier_Operational:MCP602
- added Q1, Q2: 2N7002, Package_TO_SOT_SMD:SOT-23, symbol Transistor_FET:2N7002
- added R13, R16, R17: 120k, Resistor_SMD:R_0603_1608Metric, symbol Device:R
- added R14, R15: 30k, Resistor_SMD:R_0603_1608Metric, symbol Device:R
- added R18: 51k, Resistor_SMD:R_0603_1608Metric, symbol Device:R
- added R19: 1k8, Resistor_SMD:R_0603_1608Metric, symbol Device:R
- added TP2: 3V3, TestPoint:TestPoint_THTPad_1.5x1.5mm_Drill0.7mm, symbol Connector:TestPoint
- added TP3: AmplifiedFeedback, TestPoint:TestPoint_THTPad_1.5x1.5mm_Drill0.7mm, symbol Connector:TestPoint
- added U2: TPH2504-SR, Package_SO:SOIC-14_3.9x8.7mm_P1.27mm, symbol Amplifier_Operational:LM324
- C1, C10, C5: footprint Capacitor_SMD:C_0402_1005Metric -> Capacitor_SMD:C_0603_1608Metric; LCSC C1525 -> C14663
- C11: value C -> 220p; footprint Capacitor_SMD:C_0402_1005Metric -> Capacitor_SMD:C_0603_1608Metric; LCSC (none) -> C1603
- C12: value C -> 1n5; footprint Capacitor_SMD:C_0402_1005Metric -> Capacitor_SMD:C_0603_1608Metric; LCSC (none) -> C1595
- C13: value C -> 100n; footprint Capacitor_SMD:C_0402_1005Metric -> Capacitor_SMD:C_0603_1608Metric; LCSC (none) -> C14663
- C2, C3, C4, C6, C7, C9: LCSC C19702 -> C96446
- C8: value C -> 3n3; footprint Capacitor_SMD:C_0402_1005Metric -> Capacitor_SMD:C_0603_1608Metric; LCSC (none) -> C1613
- L1: value 1u -> 1u5; footprint headlamp:MWSA0603 -> headlamp:MWSA0518; LCSC C112125 -> C408344
- R1: value 5m -> 20m; footprint Resistor_SMD:R_1206_3216Metric -> Resistor_SMD:R_0805_2012Metric; LCSC C76290 -> C92740
- R10: value R -> 3k3; LCSC (none) -> C22978
- R11, R12, R6, R8: value R -> 30k; LCSC (none) -> C22984
- R2, R3: value 10k -> 120k; LCSC (none) -> C25808
- R4: value R -> 9k1; LCSC (none) -> C23260
- R5: value R -> 91k; LCSC (none) -> C23265
- R7: value R -> 120k; LCSC (none) -> C25808
- R9: value R -> 51k; LCSC (none) -> C23196
- TP1: value FB -> ChipFeedback; footprint TestPoint:TestPoint_THTPad_1.0x1.0mm_Drill0.5mm -> TestPoint:TestPoint_THTPad_1.5x1.5mm_Drill0.7mm
- U1: LCSC (none) -> C15483
- gave numbers to parts that had none: 1
Connections:
- net +3V3: now also C13.1, R18.1, TP2.1, U2.4 (V+); no longer C12.2
- net GND: now also C13.2, R10.2, R8.2, Q1.2 (S), R17.2, R19.2, U2.11 (V-); no longer C12.1, R10.1
- net LED-: now also R12.1; no longer R6.1
- net PWM: now also R4.2; no longer R12.1
- net at NT1.1, R1.2: now also R13.1, R15.1; no longer R8.1
- net at R4.1, R5.2: now also C8.2; no longer TP1.1
- net at R6.2: now also C12.2, R5.1; no longer R8.2
- net at R9.1: now also R10.1, Q1.3 (D), U2.10 (+); no longer R10.2
- net at R11.2: now also U2.8, U2.9 (-)
- removed net DAC: C13.2, J2.11 (Pin_11), J2.12 (Pin_12), R7.1, R9.2
- new net: R7.2, TP1.1, U1.3 (FB), U2.7
- new net: R15.2, R16.1, U2.2 (-)
- new net: R12.2, R13.2, U2.3 (+)
- new net: R14.1, R16.2, U2.1
- new net: Q2.2 (S), R11.1, R14.2, TP3.1, U2.5 (+)
- new net: R7.1, R8.1, U2.6 (-)
- new net: C11.2, R6.1, U2.12 (+)
- new net: C12.1, R9.2, U2.13 (-), U2.14
- new net: Q2.3 (D), R18.2, R19.1
- new net FAST_DIM: J2.11 (Pin_11), J2.12 (Pin_12), Q1.1 (G), Q2.1 (G), R17.1
Other:
- moved on the sheet: C15, C16, J1, J2, NT1, R1, U3

Commit message: Draft first board layout
Parts:
- added H1, H2, H3, H4: MountingHole, MountingHole:MountingHole_2.2mm_M2, symbol Mechanical:MountingHole
Connections:
- net +3V3: now also U1.13 (PS/SYNC)
- net at C1.2, U1.1 (VINA): no longer U1.13 (PS/SYNC)
- net at R7.2, TP1.1, U1.3 (FB): now also U2.1; no longer U2.7
- net at R15.2, R16.1: now also U2.13 (-); no longer U2.2 (-)
- net at R12.2, R13.2: now also U2.12 (+); no longer U2.3 (+)
- net at R14.1, R16.2: now also U2.14; no longer U2.1
- net at Q2.2 (S), R11.1, R14.2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: now also U2.3 (+); no longer U2.5 (+)
- net at R7.1, R8.1: now also U2.2 (-); no longer U2.6 (-)
- net at C11.2, R6.1: now also U2.5 (+); no longer U2.12 (+)
- net at C12.1, R9.2: now also U2.6 (-), U2.7; no longer U2.13 (-), U2.14
Other:
- moved on the sheet: C1, R2, U2A, U2B, U2D
Changed lines of the file:
@@
 L Device:C C1
 U 1 1 5F22F6F4
-P 1550 2350
-F 0 "C1" H 1435 2304 50  0000 R CNN
-F 1 "100n" H 1435 2395 50  0000 R CNN
-F 2 "Capacitor_SMD:C_0603_1608Metric" H 1588 2200 50  0001 C CNN
-F 3 "~" H 1550 2350 50  0001 C CNN
-F 4 "C14663" H 1550 2350 50  0001 C CNN "LCSC"
-	1    1550 2350
+P 950 2350
+F 0 "C1" H 835 2304 50  0000 R CNN
+F 1 "100n" H 835 2395 50  0000 R CNN
+F 2 "Capacitor_SMD:C_0603_1608Metric" H 988 2200 50  0001 C CNN
+F 3 "~" H 950 2350 50  0001 C CNN
+F 4 "C14663" H 950 2350 50  0001 C CNN "LCSC"
+	1    950  2350
 	-1   0    0    1
 $EndComp
@@
 L power:GND #PWR0119
 U 1 1 5F231734
-P 1550 2500
-F 0 "#PWR0119" H 1550 2250 50  0001 C CNN
-F 1 "GND" H 1555 2327 50  0000 C CNN
-F 2 "" H 1550 2500 50  0001 C CNN
-F 3 "" H 1550 2500 50  0001 C CNN
-	1    1550 2500
+P 950 2500
+F 0 "#PWR0119" H 950 2250 50  0001 C CNN
+F 1 "GND" H 955 2327 50  0000 C CNN
+F 2 "" H 950 2500 50  0001 C CNN
+F 3 "" H 950 2500 50  0001 C CNN
+	1    950  2500
 	1    0    0    -1
 $EndComp
@@
 Wire Wire Line
 	4350 2550 4300 2550
-Wire Wire Line
-	3350 2200 3100 2200
-Wire Wire Line
-	3350 2450 3100 2450
-Wire Wire Line
-	3100 2450 3100 2200
-Connection ~ 3100 2200
-Wire Wire Line
-	3100 2200 1550 2200
 Wire Wire Line
 	3350 2550 3250 2550
@@
 L power:GND #PWR0120
 U 1 1 5F27EE89
-P 2350 2650
-F 0 "#PWR0120" H 2350 2400 50  0001 C CNN
-F 1 "GND" H 2355 2477 50  0000 C CNN
-F 2 "" H 2350 2650 50  0001 C CNN
-F 3 "" H 2350 2650 50  0001 C CNN
-	1    2350 2650
+P 1800 2650
+F 0 "#PWR0120" H 1800 2400 50  0001 C CNN
+F 1 "GND" H 1805 2477 50  0000 C CNN
+F 2 "" H 1800 2650 50  0001 C CNN
+F 3 "" H 1800 2650 50  0001 C CNN
+	1    1800 2650
 	1    0    0    -1
 $EndComp
@@
 L Device:R R2
 U 1 1 5F27F1FA
-P 2350 2500
-F 0 "R2" H 2420 2546 50  0000 L CNN
-F 1 "120k" H 2420 2455 50  0000 L CNN
-F 2 "Resistor_SMD:R_0603_1608Metric" V 2280 2500 50  0001 C CNN
-F 3 "~" H 2350 2500 50  0001 C CNN
-F 4 "C25808" H 2350 2500 50  0001 C CNN "LCSC"
-	1    2350 2500
+P 1800 2500
+F 0 "R2" H 1870 2546 50  0000 L CNN
+F 1 "120k" H 1870 2455 50  0000 L CNN
+F 2 "Resistor_SMD:R_0603_1608Metric" V 1730 2500 50  0001 C CNN
+F 3 "~" H 1800 2500 50  0001 C CNN
+F 4 "C25808" H 1800 2500 50  0001 C CNN "LCSC"
+	1    1800 2500
 	1    0    0    -1
 $EndComp
@@
 	-1   0    0    1
 $EndComp
-Wire Wire Line
-	2350 2350 3350 2350
-Text GLabel 2250 2350 0    50   Input ~ 0
+Text GLabel 1700 2350 0    50   Input ~ 0
 ENABLE
 Wire Wire Line
-	2250 2350 2350 2350
-Connection ~ 2350 2350
+	1700 2350 1800 2350
+Connection ~ 1800 2350
 Wire Wire Line
 	3700 1550 3600 1550
@@
 Text Notes 7950 1700 0    50   ~ 0
 Connect these two grounds together first and then via a single point to the rest\nof the ground. The bottom ground should be connected directly to the pad of the\nsense resistor.
-$Comp
-L Device:Net-Tie_2 NT1
-U 1 1 5F3732B0
-P 8850 1950
-F 0 "NT1" H 8850 2131 50  0000 C CNN
-F 1 "SenseTie" H 8850 2040 50  0000 C CNN
-F 2 "NetTie:NetTie-2_SMD_Pad0.5mm" H 8850 1950 50  0001 C CNN
-F 3 "~" H 8850 1950 50  0001 C CNN
-	1    8850 1950
-	1    0    0    -1
-$EndComp
 Wire Wire Line
 	9100 1950 8950 1950
@@
 L Amplifier_Operational:LM324 U2
 U 1 1 5F35AF0D
-P 7550 2750
-F 0 "U2" V 7500 3100 50  0000 R CNN
-F 1 "TPH2504-SR" V 7600 3400 50  0000 R CNN
-F 2 "Package_SO:SOIC-14_3.9x8.7mm_P1.27mm" H 7500 2850 50  0001 C CNN
-F 3 "http://www.ti.com/lit/ds/symlink/lm2902-n.pdf" H 7600 2950 50  0001 C CNN
-F 4 "C115918" H 7550 2750 50  0001 C CNN "LCSC"
-	1    7550 2750
-	0    -1   1    0
-$EndComp
-$Comp
-L Amplifier_Operational:LM324 U2
-U 2 1 5F35C47E
 P 6100 3200
-F 0 "U2" H 6100 3567 50  0000 C CNN
-F 1 "TPH2504-SR" H 6100 3476 50  0000 C CNN
+F 0 "U2" V 6050 3550 50  0000 R CNN
+F 1 "TPH2504-SR" V 6150 3850 50  0000 R CNN
 F 2 "Package_SO:SOIC-14_3.9x8.7mm_P1.27mm" H 6050 3300 50  0001 C CNN
 F 3 "http://www.ti.com/lit/ds/symlink/lm2902-n.pdf" H 6150 3400 50  0001 C CNN
 F 4 "C115918" H 6100 3200 50  0001 C CNN "LCSC"
-	2    6100 3200
+	1    6100 3200
 	-1   0    0    -1
+$EndComp
+$Comp
+L Amplifier_Operational:LM324 U2
+U 2 1 5F35C47E
+P 5850 4900
+F 0 "U2" H 5850 5200 50  0000 C CNN
+F 1 "TPH2504-SR" H 6050 5100 50  0000 C CNN
+F 2 "Package_SO:SOIC-14_3.9x8.7mm_P1.27mm" H 5800 5000 50  0001 C CNN
+F 3 "http://www.ti.com/lit/ds/symlink/lm2902-n.pdf" H 5900 5100 50  0001 C CNN
+F 4 "C115918" H 5850 4900 50  0001 C CNN "LCSC"
+	2    5850 4900
+	1    0    0    -1
 $EndComp
 $Comp
@@
 $Comp
 L Amplifier_Operational:LM324 U2
-U 4 1 5F35F1E1
-P 5850 4900
-F 0 "U2" H 5900 5200 50  0000 C CNN
-F 1 "TPH2504-SR" H 6050 5100 50  0000 C CNN
-F 2 "Package_SO:SOIC-14_3.9x8.7mm_P1.27mm" H 5800 5000 50  0001 C CNN
-F 3 "http://www.ti.com/lit/ds/symlink/lm2902-n.pdf" H 5900 5100 50  0001 C CNN
-F 4 "C115918" H 5850 4900 50  0001 C CNN "LCSC"
-	4    5850 4900
-	1    0    0    -1
-$EndComp
-$Comp
-L Amplifier_Operational:LM324 U2
 U 5 1 5F361281
 P 5850 4900
@@
 	1    0    0    -1
 $EndComp
-Connection ~ 7550 3050
 Wire Wire Line
 	7550 3450 7350 3450
@@
 Wire Wire Line
 	7900 1950 8050 1950
+$Comp
+L Device:Net-Tie_2 NT1
+U 1 1 5F3732B0
+P 8850 1950
+F 0 "NT1" H 8850 2131 50  0000 C CNN
+F 1 "SenseTie" H 8850 2040 50  0000 C CNN
+F 2 "NetTie:NetTie-2_SMD_Pad0.5mm" H 8850 1950 50  0001 C CNN
+F 3 "~" H 8850 1950 50  0001 C CNN
+	1    8850 1950
+	1    0    0    -1
+$EndComp
+$Comp
+L Amplifier_Operational:LM324 U2
+U 4 1 5F35F1E1
+P 7550 2750
+F 0 "U2" H 7600 3050 50  0000 C CNN
+F 1 "TPH2504-SR" H 7750 2950 50  0000 C CNN
+F 2 "Package_SO:SOIC-14_3.9x8.7mm_P1.27mm" H 7500 2850 50  0001 C CNN
+F 3 "http://www.ti.com/lit/ds/symlink/lm2902-n.pdf" H 7600 2950 50  0001 C CNN
+F 4 "C115918" H 7550 2750 50  0001 C CNN "LCSC"
+	4    7550 2750
+	0    -1   1    0
+$EndComp
+Connection ~ 7550 3050
+$Comp
+L Mechanical:MountingHole H3
+U 1 1 5F812976
+P 1300 5050
+F 0 "H3" H 1400 5096 50  0000 L CNN
+F 1 "MountingHole" H 1400 5005 50  0000 L CNN
+F 2 "MountingHole:MountingHole_2.2mm_M2" H 1300 5050 50  0001 C CNN
+F 3 "~" H 1300 5050 50  0001 C CNN
+	1    1300 5050
+	1    0    0    -1
+$EndComp
+$Comp
+L Mechanical:MountingHole H4
+U 1 1 5F812F86
+P 1300 5250
+F 0 "H4" H 1400 5296 50  0000 L CNN
+F 1 "MountingHole" H 1400 5205 50  0000 L CNN
+F 2 "MountingHole:MountingHole_2.2mm_M2" H 1300 5250 50  0001 C CNN
+F 3 "~" H 1300 5250 50  0001 C CNN
+	1    1300 5250
+	1    0    0    -1
+$EndComp
+$Comp
+L Mechanical:MountingHole H1
+U 1 1 5F815CE7
+P 1300 4600
+F 0 "H1" H 1400 4646 50  0000 L CNN
+F 1 "MountingHole" H 1400 4555 50  0000 L CNN
+F 2 "MountingHole:MountingHole_2.2mm_M2" H 1300 4600 50  0001 C CNN
+F 3 "~" H 1300 4600 50  0001 C CNN
+	1    1300 4600
+	1    0    0    -1
+$EndComp
+$Comp
+L Mechanical:MountingHole H2
+U 1 1 5F815CED
+P 1300 4800
+F 0 "H2" H 1400 4846 50  0000 L CNN
+F 1 "MountingHole" H 1400 4755 50  0000 L CNN
+F 2 "MountingHole:MountingHole_2.2mm_M2" H 1300 4800 50  0001 C CNN
+F 3 "~" H 1300 4800 50  0001 C CNN
+	1    1300 4800
+	1    0    0    -1
+$EndComp
+Wire Wire Line
+	950  2200 3350 2200
+Wire Wire Line
+	1800 2350 3350 2350
+$Comp
+L power:+3.3V #PWR?
+U 1 1 5F85B2BF
+P 2300 2450
+F 0 "#PWR?" H 2300 2300 50  0001 C CNN
+F 1 "+3.3V" H 2315 2623 50  0000 C CNN
+F 2 "" H 2300 2450 50  0001 C CNN
+F 3 "" H 2300 2450 50  0001 C CNN
+	1    2300 2450
+	-1   0    0    1
+$EndComp
+Wire Wire Line
+	2300 2450 3350 2450
 $EndSCHEMATC

Commit message: Tweak assembly data
Parts:
- Q1, Q2, U3: JLCPCB_CORRECTION (none) -> 0;0;180
- U2: JLCPCB_CORRECTION (none) -> 0;0;-90
Changed lines of the file:
@@
 F 3 "https://www.torexsemi.com/file/xc6206/XC6206.pdf" H 4650 6550 50  0001 C CNN
 F 4 "C5446" H 4650 6550 50  0001 C CNN "LCSC"
+F 5 "0;0;180" H 4650 6550 50  0001 C CNN "JLCPCB_CORRECTION"
 	1    4650 6550
 	1    0    0    -1
@@
 F 3 "http://www.ti.com/lit/ds/symlink/lm2902-n.pdf" H 6150 3400 50  0001 C CNN
 F 4 "C115918" H 6100 3200 50  0001 C CNN "LCSC"
+F 5 "0;0;-90" H 6100 3200 50  0001 C CNN "JLCPCB_CORRECTION"
 	1    6100 3200
 	-1   0    0    -1
@@
 F 3 "http://www.ti.com/lit/ds/symlink/lm2902-n.pdf" H 5900 5100 50  0001 C CNN
 F 4 "C115918" H 5850 4900 50  0001 C CNN "LCSC"
+F 5 "0;0;-90" H 5850 4900 50  0001 C CNN "JLCPCB_CORRECTION"
 	2    5850 4900
 	1    0    0    -1
@@
 F 3 "http://www.ti.com/lit/ds/symlink/lm2902-n.pdf" H 7050 4500 50  0001 C CNN
 F 4 "C115918" H 7000 4300 50  0001 C CNN "LCSC"
+F 5 "0;0;-90" H 7000 4300 50  0001 C CNN "JLCPCB_CORRECTION"
 	3    7000 4300
 	0    -1   -1   0
@@
 F 3 "http://www.ti.com/lit/ds/symlink/lm2902-n.pdf" H 5900 5100 50  0001 C CNN
 F 4 "C115918" H 5850 4900 50  0001 C CNN "LCSC"
+F 5 "0;0;-90" H 5850 4900 50  0001 C CNN "JLCPCB_CORRECTION"
 	5    5850 4900
 	1    0    0    -1
@@
 F 3 "https://www.fairchildsemi.com/datasheets/2N/2N7002.pdf" H 7700 5150 50  0001 L CNN
 F 4 "C8545" H 7700 5150 50  0001 C CNN "LCSC"
+F 5 "0;0;180" H 7700 5150 50  0001 C CNN "JLCPCB_CORRECTION"
 	1    7700 5150
 	-1   0    0    -1
@@
 F 3 "https://www.fairchildsemi.com/datasheets/2N/2N7002.pdf" H 8400 4950 50  0001 L CNN
 F 4 "C8545" H 8400 4950 50  0001 C CNN "LCSC"
+F 5 "0;0;180" H 8400 4950 50  0001 C CNN "JLCPCB_CORRECTION"
 	1    8400 4950
 	0    1    -1   0
@@
 	8400 5450 8400 5800
 Wire Wire Line
-	8400 5800 3450 5750
+	8400 5800 3450 5800
 Connection ~ 8400 5450
-Text GLabel 3450 5750 0    50   Input ~ 0
+Text GLabel 3450 5800 0    50   Input ~ 0
 FAST_DIM
 Text GLabel 1950 7250 0    50   Input ~ 0
@@
 F 3 "http://www.ti.com/lit/ds/symlink/lm2902-n.pdf" H 7600 2950 50  0001 C CNN
 F 4 "C115918" H 7550 2750 50  0001 C CNN "LCSC"
+F 5 "0;0;-90" H 7550 2750 50  0001 C CNN "JLCPCB_CORRECTION"
 	4    7550 2750
 	0    -1   1    0
@@
 	1800 2350 3350 2350
 $Comp
-L power:+3.3V #PWR?
+L power:+3.3V #PWR0106
 U 1 1 5F85B2BF
 P 2300 2450
-F 0 "#PWR?" H 2300 2300 50  0001 C CNN
+F 0 "#PWR0106" H 2300 2300 50  0001 C CNN
 F 1 "+3.3V" H 2315 2623 50  0000 C CNN
 F 2 "" H 2300 2450 50  0001 C CNN
